File: OpenAmiga2000CoproAdapter.sch (KiCad schematic (older format))
At the start: 18 parts, among them CN1 A2000_COPRO_SLOT, P1 CONN_2, P10 CONN_1, P11 CONN_1, P12 CONN_1, P13 CONN_1, P14 CONN_1, P15 CONN_1, P2 CONN_2, P3 CONN_2, P4 CONN_2, P5 CONN_1, P6 CONN_1, P7 CONN_1, P8 CONN_1, P9 CONN_1, P99 OSHW_LOGO, U1 68000D

Commit message: Experiment arbitrating bus away from mainboard cpu
Parts:
- removed P12: CONN_1, TestPoint:TestPoint_Pad_D1.5mm, symbol conn:CONN_1
- added C1, C2: C, Capacitor_SMD:C_0805_2012Metric_Pad1.15x1.40mm_HandSolder, symbol Device:C
- added JP1: SolderJumper_3_Bridged12, Jumper:SolderJumper-3_P1.3mm_Bridged12_RoundedPad1.0x1.5mm, symbol Jumper:SolderJumper_3_Bridged12
- added JP2: SolderJumper_2_Open, Jumper:SolderJumper-2_P1.3mm_Open_RoundedPad1.0x1.5mm, symbol Jumper:SolderJumper_2_Open
- added Q1, Q2, Q3, Q4, Q5, Q6, Q7: 2N7002, Package_TO_SOT_SMD:SOT-23, symbol Transistor_FET:2N7002
- added U2: 74HC74, Package_SO:SOIC-14_3.9x8.7mm_P1.27mm, symbol 74xx:74HC74
- added U3: 74HC00, Package_SO:SOIC-14_3.9x8.7mm_P1.27mm, symbol 74xx:74HC00
- P1, P2, P3, P4: symbol conn:CONN_2 -> OpenAmiga2000CoproAdapter-rescue:CONN_2-conn
- P10, P11, P13, P14, P15, P5, P6, P7, P8, P9, P99: symbol conn:CONN_1 -> OpenAmiga2000CoproAdapter-rescue:CONN_1-conn
Connections:
- net labels added: BR, ~BOSS, ~BR, ~cpuhlt, ~cpurst
- wire segments 186 -> 230
- no-connect marks 1 -> 2
Other:
- note added: "Arbitrate bus away from mainboard CPU\nKeeps coprocessor in reset and isolates it's halt + reset until BG is asserted then we assert BOSS and release BR"
- note added: "OFF"
- note added: "ON"
