File: OpenAmiga2000CoproAdapter.kicad_sch (KiCad schematic)
At the start: 39 parts, among them CN1 A2000_COPRO_SLOT, J1 Conn_01x06_Male, P10 CONN_1, P11 CONN_1, P12 CONN_1, P13 CONN_1, P14 CONN_1, P15 CONN_1, P16 CONN_1, P17 CONN_2, P5 CONN_2, P6 OSHW_LOGO, P7 CONN_1, P8 CONN_1, P9 CONN_1, U1 68000D, U2 AP2210N-3.3, U3 XC9572VQ44, U4 74CBTD3306

Commit message: Boss proto stuff
Connections:
- net ~a_hlt: no longer U4.3 (1B)
- net ~a_lds: now also JP7.2 (B); no longer JP8.2 (B)
- net ~a_rst: no longer U4.6 (2B)
- net ~a_uds: now also JP8.2 (B); no longer JP7.2 (B)
Other:
- note added: "CPLD isolates the following signals until BOSS asseted. could be replaced by some 74CBT buffer instead BR BG RW LDS UDS AS* BG* BR* FC0-2 * = Also Used by CPLD Logic"
- note added: "Jumpers to bypass CPLD"
- note added: "RESET/HALT isolated until BOSS active This allows the CPLD to hold the "coprocessor" in reset without affecting the Amiga"
- moved on the sheet: C1, C2, C6, U2, U4
